File: AXremote_circuit/remote.sch (EAGLE design)
At the start: 22 parts, among them Q1 16MHz, U1 AX8052F143HS

Commit message: ...
Other:
- note added: "not necessary: - RX/TX - PB3"
- note added: "todo: - buttons (matrix, shift reg, ..?) - battery measurement - low power led - status (tx)/debug led - battery, ev. regulator, ev. buffer (C)? - on/off switch"
- note removed: "todo: - buttons (matrix, shift reg, ..?) - battery measurement - low power led - status (tx)/debug led - battery, ev. regulator - on/off switch"
Changed lines of the file:
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@@
 - low power led
 - status (tx)/debug led
-- battery, ev. regulator
+- battery, ev. regulator, ev. buffer (C)?
 - on/off switch</text>
+<text x="81.28" y="-17.78" size="1.778" layer="91">not necessary:
+- RX/TX
+- PB3</text>
 </plain>
 <instances>
@@
 <wire x1="-177.8" y1="10.16" x2="-203.2" y2="10.16" width="0.1524" layer="91"/>
 <wire x1="-203.2" y1="10.16" x2="-203.2" y2="15.24" width="0.1524" layer="91"/>
-<wire x1="-203.2" y1="15.24" x2="-165.1" y2="15.24" width="0.1524" layer="91"/>
+<wire x1="-203.2" y1="15.24" x2="-185.42" y2="15.24" width="0.1524" layer="91"/>
 <wire x1="-203.2" y1="-20.32" x2="-203.2" y2="-25.4" width="0.1524" layer="91"/>
 <wire x1="-203.2" y1="-25.4" x2="-157.48" y2="-25.4" width="0.1524" layer="91"/>

Commit message: remote almost complete
Parts:
- added C1: 100uF, resistor:CPOL-EUE
- added C2: 100uF, resistor:C-EUC1206K
- added JP1: (no value), pinhead:PINHD-1X2
- added LED1, LED2: (no value), led:LEDCHIPLED_1206
- added R1, R3: (no value), resistor:R-EU_R0603
- added S1, S10, S11, S12, S13, S14, S15, S16, S17, S18, S19, S2, S20, S21, S22, S23, S24, S25, S28, S3, S30, S4, S41, S42, S43, S44, S45, S46, S5, S6, S7, S8, S9: (no value), switch-omron:10-XX
- added U$2: 2X5PIN-CONNECTOR, sam_eagle_parts:2X5PIN-CONNECTOR
- C10, C4, C5: device resistor:C-EUC1206 -> resistor:C-EUC0603
- U$1: value PINHEADER5X2 -> CR2032; device sam:PINHEADER5X2 -> sam_eagle_parts:CR2032
Connections:
- removed net BATTMEASURE: U1IC.PA0
- removed net RX0: U$1.P$7, U1IC.PB5
- removed net TX0: U$1.P$8, U1IC.PB4
- new net COL0: S1.S, S1.S1, S11.S, S11.S1, S16.S, S16.S1, S21.S, S21.S1, S6.S, S6.S1, U1IC.PB5
- new net COL1: S12.S, S12.S1, S17.S, S17.S1, S2.S, S2.S1, S22.S, S22.S1, S7.S, S7.S1, U1IC.PB4
- new net COL2: S13.S, S13.S1, S18.S, S18.S1, S23.S, S23.S1, S28.S, S28.S1, S3.S, S3.S1, S8.S, S8.S1, U1IC.PB3
- new net COL3: S14.S, S14.S1, S19.S, S19.S1, S24.S, S24.S1, S4.S, S4.S1, S9.S, S9.S1, U1IC.PB2
- new net COL4: S10.S, S10.S1, S15.S, S15.S1, S20.S, S20.S1, S25.S, S25.S1, S30.S, S30.S1, S5.S, S5.S1, U1IC.PB1
- new net COL5: S41.S, S41.S1, S42.S, S42.S1, S43.S, S43.S1, S44.S, S44.S1, S45.S, S45.S1, S46.S, S46.S1, U1IC.PB0
- new net N$11: LED2.A, U1IC.PA5
- new net N$17: LED1.C, R1.2
- new net N$4: LED1.A, U1IC.PA4
- new net N$64: C1.+, C2.1, JP1.1, U$1.P$PLUS
- new net ROW0: S1.P, S1.P1, S2.P, S2.P1, S3.P, S3.P1, S4.P, S4.P1, S41.P, S41.P1, S5.P, S5.P1, U1IC.PC0
- new net ROW1: S10.P, S10.P1, S42.P, S42.P1, S6.P, S6.P1, S7.P, S7.P1, S8.P, S8.P1, S9.P, S9.P1, U1IC.PC1
- new net ROW2: S11.P, S11.P1, S12.P, S12.P1, S13.P, S13.P1, S14.P, S14.P1, S15.P, S15.P1, S43.P, S43.P1, U1IC.PC2
- new net ROW3: S16.P, S16.P1, S17.P, S17.P1, S18.P, S18.P1, S19.P, S19.P1, S20.P, S20.P1, S44.P, S44.P1, U1IC.PC3
- new net ROW4: S21.P, S21.P1, S22.P, S22.P1, S23.P, S23.P1, S24.P, S24.P1, S25.P, S25.P1, S45.P, S45.P1, U1IC.PC4
- new net ROW5: S28.P, S28.P1, S30.P, S30.P1, S46.P, S46.P1, U1IC.PA0
- new net ROW6: U1IC.PA1
- new net ROW7: U1IC.PA2
- new net ROW8: U1IC.PA3
- net DBG_CLK: now also U$2.P$5; no longer U$1.P$5
- net DBG_DATA: now also U$2.P$6; no longer U$1.P$6
- net DBG_EN: now also U$2.P$4; no longer U$1.P$4
- net GND: now also C1.-, C2.2, R1.1, R3.1, U$1.P$MINUS, U$2.P$10, U$2.P$2; no longer U$1.P$10, U$1.P$2
- net N$16: now also LED2.C, R3.2; no longer U$1.P$9, U1IC.PB3
- net N$5: now also U$2.P$3; no longer U$1.P$3
- net VCC: now also JP1.2, U$2.P$1; no longer U$1.P$1
Other:
- note removed: "not necessary: - RX/TX - PB3"
- moved on the sheet: U1GP

Commit message: Remote and receiver done.
Parts:
- added U$3: APERTURE_LOGO, sam_eagle_parts:APERTURE_LOGO
Changed lines of the file:
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@@
 <layers>
 <layer number="1" name="Top" color="4" fill="1" visible="no" active="no"/>
+<layer number="2" name="Route2" color="1" fill="3" visible="no" active="no"/>
+<layer number="3" name="Route3" color="4" fill="3" visible="no" active="no"/>
+<layer number="4" name="Route4" color="1" fill="4" visible="no" active="no"/>
+<layer number="5" name="Route5" color="4" fill="4" visible="no" active="no"/>
+<layer number="6" name="Route6" color="1" fill="8" visible="no" active="no"/>
+<layer number="7" name="Route7" color="4" fill="8" visible="no" active="no"/>
+<layer number="8" name="Route8" color="1" fill="2" visible="no" active="no"/>
+<layer number="9" name="Route9" color="4" fill="2" visible="no" active="no"/>
+<layer number="10" name="Route10" color="1" fill="7" visible="no" active="no"/>
+<layer number="11" name="Route11" color="4" fill="7" visible="no" active="no"/>
+<layer number="12" name="Route12" color="1" fill="5" visible="no" active="no"/>
+<layer number="13" name="Route13" color="4" fill="5" visible="no" active="no"/>
+<layer number="14" name="Route14" color="1" fill="6" visible="no" active="no"/>
+<layer number="15" name="Route15" color="4" fill="6" visible="no" active="no"/>
 <layer number="16" name="Bottom" color="1" fill="1" visible="no" active="no"/>
 <layer number="17" name="Pads" color="2" fill="1" visible="no" active="no"/>
@@
 <part name="S45" library="switch-omron" deviceset="10-XX" device=""/>
 <part name="S46" library="switch-omron" deviceset="10-XX" device=""/>
+<part name="U$3" library="sam_eagle_parts" deviceset="APERTURE_LOGO" device=""/>
 </parts>
 <sheets>
@@
 <instance part="S45" gate="1" x="314.96" y="-86.36" rot="R270"/>
 <instance part="S46" gate="1" x="314.96" y="-116.84" rot="R270"/>
+<instance part="U$3" gate="G$1" x="-101.6" y="45.72"/>
 </instances>
 <busses>
@@
 <pinref part="S41" gate="1" pin="P1"/>
 <wire x1="307.34" y1="33.02" x2="309.88" y2="33.02" width="0.1524" layer="91"/>
+<junction x="193.04" y="33.02"/>
+<junction x="215.9" y="33.02"/>
+<junction x="238.76" y="33.02"/>
+<junction x="307.34" y="33.02"/>
+<junction x="284.48" y="33.02"/>
+<junction x="261.62" y="33.02"/>
 </segment>
 <segment>
@@
 <wire x1="208.28" y1="-119.38" x2="205.74" y2="-119.38" width="0.1524" layer="91"/>
 <junction x="208.28" y="-116.84"/>
+<junction x="208.28" y="33.02"/>
+<junction x="208.28" y="-88.9"/>
+<junction x="208.28" y="2.54"/>
 </segment>
 <segment>
@@
 <wire x1="231.14" y1="-119.38" x2="228.6" y2="-119.38" width="0.1524" layer="91"/>
 <junction x="231.14" y="-116.84"/>
+<junction x="231.14" y="-88.9"/>
+<junction x="231.14" y="2.54"/>
+<junction x="231.14" y="33.02"/>
 </segment>
 <segment>
@@
 <wire x1="254" y1="-119.38" x2="251.46" y2="-119.38" width="0.1524" layer="91"/>
 <junction x="254" y="-116.84"/>
+<junction x="254" y="2.54"/>
+<junction x="254" y="33.02"/>
+<junction x="254" y="-88.9"/>
 </segment>
 <segment>
@@
 <wire x1="276.86" y1="-119.38" x2="274.32" y2="-119.38" width="0.1524" layer="91"/>
 <junction x="276.86" y="-116.84"/>
+<junction x="276.86" y="2.54"/>
+<junction x="276.86" y="33.02"/>
+<junction x="276.86" y="-88.9"/>
 </segment>
 <segment>
@@
 <wire x1="299.72" y1="-119.38" x2="297.18" y2="-119.38" width="0.1524" layer="91"/>
 <junction x="299.72" y="-116.84"/>
+<junction x="299.72" y="2.54"/>
+<junction x="299.72" y="33.02"/>
+<junction x="299.72" y="-88.9"/>
 </segment>
 <segment>
@@
 <pinref part="S9" gate="1" pin="P1"/>
 <wire x1="264.16" y1="2.54" x2="261.62" y2="2.54" width="0.1524" layer="91"/>
+<junction x="215.9" y="2.54"/>
+<junction x="193.04" y="2.54"/>
+<junction x="238.76" y="2.54"/>
+<junction x="261.62" y="2.54"/>
+<junction x="284.48" y="2.54"/>
+<junction x="307.34" y="2.54"/>
 </segment>
 <segment>
@@
 <pinref part="S45" gate="1" pin="P1"/>
 <wire x1="307.34" y1="-88.9" x2="309.88" y2="-88.9" width="0.1524" layer="91"/>
+<junction x="193.04" y="-88.9"/>
+<junction x="215.9" y="-88.9"/>
+<junction x="238.76" y="-88.9"/>
+<junction x="261.62" y="-88.9"/>
+<junction x="284.48" y="-88.9"/>
+<junction x="307.34" y="-88.9"/>
 </segment>
 <segment>
@@
 <wire x1="322.58" y1="-119.38" x2="320.04" y2="-119.38" width="0.1524" layer="91"/>
 <junction x="322.58" y="-116.84"/>
-</segment>
-<segment>
+<junction x="322.58" y="2.54"/>
+<junction x="322.58" y="33.02"/>
+<junction x="322.58" y="-88.9"/>
+</segment>
+<segment>
