File: AXremote_circuit/remote.sch (EAGLE design)
At the start: 64 parts, among them Q1 16MHz, U1 AX8052F143HS

Commit message: Added a few keys.
Parts:
- added R4: (no value), resistor:R-EU_R0603
Connections:
- removed net N$64: C1.+, C2.1, JP1.1, U$1.P$PLUS
- new net N$18: C1.+, C2.1, JP1.1, R4.2, U$1.P$PLUS
- net N$5: now also R4.1
Changed lines of the file:
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@@
 <?xml version="1.0" encoding="utf-8"?>
 <!DOCTYPE eagle SYSTEM "eagle.dtd">
-<eagle version="6.4">
+<eagle version="6.5.0">
 <drawing>
 <settings>
@@
 <part name="S46" library="switch-omron" deviceset="10-XX" device=""/>
 <part name="U$3" library="sam_eagle_parts" deviceset="APERTURE_LOGO" device=""/>
+<part name="R4" library="resistor" deviceset="R-EU_" device="R0603"/>
 </parts>
 <sheets>
@@
 <instance part="S46" gate="1" x="314.96" y="-116.84" rot="R270"/>
 <instance part="U$3" gate="G$1" x="-101.6" y="45.72"/>
+<instance part="R4" gate="G$1" x="63.5" y="15.24"/>
 </instances>
 <busses>
@@
 <wire x1="73.66" y1="0" x2="63.5" y2="0" width="0.1524" layer="91"/>
 <wire x1="63.5" y1="0" x2="63.5" y2="5.08" width="0.1524" layer="91"/>
-<wire x1="63.5" y1="5.08" x2="27.94" y2="5.08" width="0.1524" layer="91"/>
+<wire x1="63.5" y1="5.08" x2="55.88" y2="5.08" width="0.1524" layer="91"/>
 <pinref part="U$2" gate="G$1" pin="P$3"/>
+<pinref part="R4" gate="G$1" pin="1"/>
+<wire x1="55.88" y1="5.08" x2="27.94" y2="5.08" width="0.1524" layer="91"/>
+<wire x1="58.42" y1="15.24" x2="55.88" y2="15.24" width="0.1524" layer="91"/>
+<wire x1="55.88" y1="15.24" x2="55.88" y2="5.08" width="0.1524" layer="91"/>
+<junction x="55.88" y="5.08"/>
 </segment>
 </net>
@@
 </segment>
 </net>
-<net name="N$64" class="0">
-<segment>
-<pinref part="C2" gate="G$1" pin="1"/>
-<wire x1="99.06" y1="43.18" x2="101.6" y2="43.18" width="0.1524" layer="91"/>
-<wire x1="101.6" y1="43.18" x2="101.6" y2="50.8" width="0.1524" layer="91"/>
-<pinref part="C1" gate="G$1" pin="+"/>
-<wire x1="101.6" y1="50.8" x2="101.6" y2="68.58" width="0.1524" layer="91"/>
-<wire x1="99.06" y1="50.8" x2="101.6" y2="50.8" width="0.1524" layer="91"/>
-<wire x1="101.6" y1="50.8" x2="111.76" y2="50.8" width="0.1524" layer="91"/>
-<pinref part="JP1" gate="G$1" pin="1"/>
-<wire x1="111.76" y1="58.42" x2="111.76" y2="50.8" width="0.1524" layer="91"/>
-<pinref part="U$1" gate="G$1" pin="P$PLUS"/>
-<junction x="101.6" y="50.8"/>
-</segment>
-</net>
 <net name="N$4" class="0">
 <segment>
@@
 </segment>
 </net>
+<net name="N$18" class="0">
+<segment>
+<pinref part="R4" gate="G$1" pin="2"/>
+<pinref part="C2" gate="G$1" pin="1"/>
+<wire x1="99.06" y1="43.18" x2="101.6" y2="43.18" width="0.1524" layer="91"/>
+<wire x1="101.6" y1="43.18" x2="101.6" y2="50.8" width="0.1524" layer="91"/>
+<pinref part="C1" gate="G$1" pin="+"/>
+<wire x1="101.6" y1="50.8" x2="101.6" y2="68.58" width="0.1524" layer="91"/>
+<wire x1="99.06" y1="50.8" x2="101.6" y2="50.8" width="0.1524" layer="91"/>
+<wire x1="101.6" y1="50.8" x2="111.76" y2="50.8" width="0.1524" layer="91"/>
+<pinref part="JP1" gate="G$1" pin="1"/>
+<wire x1="111.76" y1="58.42" x2="111.76" y2="50.8" width="0.1524" layer="91"/>
+<pinref part="U$1" gate="G$1" pin="P$PLUS"/>
+<junction x="101.6" y="50.8"/>
+<wire x1="68.58" y1="15.24" x2="111.76" y2="15.24" width="0.1524" layer="91"/>
+<wire x1="111.76" y1="15.24" x2="111.76" y2="50.8" width="0.1524" layer="91"/>
+<junction x="111.76" y="50.8"/>
+</segment>
+</net>

Commit message: Start rev 3, full SMD.
Parts:
- removed JP1: (no value), pinhead:PINHD-1X2
- removed S41, S42, S43, S44, S45, S46: (no value), switch-omron:10-XX
- added S26, S27, S29, S31, S32, S34: SWITCHSMD, sam:SWITCHSMD
- S1, S10, S11, S12, S13, S14, S15, S16, S17, S18, S19, S2, S20, S21, S22, S23, S24, S25, S28, S3, S30, S4, S5, S6, S7, S8, S9: value (none) -> SWITCHSMD; device switch-omron:10-XX -> sam:SWITCHSMD
Connections:
- removed net N$18: C1.+, C2.1, JP1.1, R4.2, U$1.P$PLUS
- new net ROW10: S16.P3
- new net ROW11: S22.P3
- new net ROW12: S28.P3
- new net ROW13: S34.P3
- new net ROW9: S10.P3
- net COL0: now also S1.P1, S1.P2; no longer S1.S, S1.S1, S11.S, S11.S1, S16.S, S16.S1, S21.S, S21.S1, S6.S, S6.S1
- net COL1: now also S2.P1, S2.P2; no longer S12.S, S12.S1, S17.S, S17.S1, S2.S, S2.S1, S22.S, S22.S1, S7.S, S7.S1
- net COL2: now also S3.P1, S3.P2; no longer S13.S, S13.S1, S18.S, S18.S1, S23.S, S23.S1, S28.S, S28.S1, S3.S, S3.S1, S8.S, S8.S1
- net COL3: now also S4.P1, S4.P2; no longer S14.S, S14.S1, S19.S, S19.S1, S24.S, S24.S1, S4.S, S4.S1, S9.S, S9.S1
- net COL4: now also S5.P1, S5.P2; no longer S10.S, S10.S1, S15.S, S15.S1, S20.S, S20.S1, S25.S, S25.S1, S30.S, S30.S1, S5.S, S5.S1
- net COL5: now also S6.P1, S6.P2; no longer S41.S, S41.S1, S42.S, S42.S1, S43.S, S43.S1, S44.S, S44.S1, S45.S, S45.S1, S46.S, S46.S1
- net ROW0: now also S1.P3, S1.P4, S2.P3, S2.P4, S3.P3, S3.P4, S4.P3, S4.P4, S5.P3, S5.P4, S6.P3, S6.P4; no longer S1.P, S1.P1, S2.P, S2.P1, S3.P, S3.P1, S4.P, S4.P1, S41.P, S41.P1, S5.P, S5.P1
- net ROW1: no longer S10.P, S10.P1, S42.P, S42.P1, S6.P, S6.P1, S7.P, S7.P1, S8.P, S8.P1, S9.P, S9.P1
- net ROW2: no longer S11.P, S11.P1, S12.P, S12.P1, S13.P, S13.P1, S14.P, S14.P1, S15.P, S15.P1, S43.P, S43.P1
- net ROW3: no longer S16.P, S16.P1, S17.P, S17.P1, S18.P, S18.P1, S19.P, S19.P1, S20.P, S20.P1, S44.P, S44.P1
- net ROW4: no longer S21.P, S21.P1, S22.P, S22.P1, S23.P, S23.P1, S24.P, S24.P1, S25.P, S25.P1, S45.P, S45.P1
- net ROW5: no longer S28.P, S28.P1, S30.P, S30.P1, S46.P, S46.P1
- net VCC: now also C1.+, C2.1, R4.2, U$1.P$PLUS; no longer JP1.2

Commit message: Routed rev4, all SMD.
Parts:
- removed U$1: CR2032, sam_eagle_parts:CR2032
- removed U$3: APERTURE_LOGO, sam_eagle_parts:APERTURE_LOGO
- added BATTERY: BATTERYSMD, sam:BATTERYSMD
- added L7: (no value), SparkFun-Passives:INDUCTORNPI75
- R4: value (none) -> 10k
Connections:
- removed net ROW10: S16.P3
- removed net ROW11: S22.P3
- removed net ROW12: S28.P3
- removed net ROW13: S34.P3
- removed net ROW9: S10.P3
- new net N$18: BATTERY.PLUS, L7.1
- net COL0: now also S13.P1, S13.P2, S19.P1, S19.P2, S25.P1, S25.P2, S31.P1, S31.P2, S7.P1, S7.P2
- net COL1: now also S14.P1, S14.P2, S20.P1, S20.P2, S26.P1, S26.P2, S32.P1, S32.P2, S8.P1, S8.P2
- net COL2: now also S15.P1, S15.P2, S21.P1, S21.P2, S27.P1, S27.P2, S9.P1, S9.P2
- net COL3: now also S10.P1, S10.P2, S16.P1, S16.P2, S22.P1, S22.P2, S28.P1, S28.P2, S34.P1, S34.P2
- net COL4: now also S11.P1, S11.P2, S17.P1, S17.P2, S23.P1, S23.P2, S29.P1, S29.P2
- net COL5: now also S12.P1, S12.P2, S18.P1, S18.P2, S24.P1, S24.P2, S30.P1, S30.P2
- net GND: now also BATTERY.MINUS; no longer U$1.P$MINUS
- net ROW1: now also S10.P3, S10.P4, S11.P3, S11.P4, S12.P3, S12.P4, S7.P3, S7.P4, S8.P3, S8.P4, S9.P3, S9.P4
- net ROW2: now also S13.P3, S13.P4, S14.P3, S14.P4, S15.P3, S15.P4, S16.P3, S16.P4, S17.P3, S17.P4, S18.P3, S18.P4
- net ROW3: now also S19.P3, S19.P4, S20.P3, S20.P4, S21.P3, S21.P4, S22.P3, S22.P4, S23.P3, S23.P4, S24.P3, S24.P4
- net ROW4: now also S25.P3, S25.P4, S26.P3, S26.P4, S27.P3, S27.P4, S28.P3, S28.P4, S29.P3, S29.P4, S30.P3, S30.P4
- net ROW5: now also S31.P3, S31.P4, S32.P3, S32.P4, S34.P3, S34.P4
- net VCC: now also L7.2; no longer U$1.P$PLUS
