File: AXremote_circuit/remote.brd (EAGLE design)
At the start: 240 x 49 mm, 89 parts, among them Q1 16MHz, U1 AX8052F143HS

Commit message: GND polygon thicker, fix typo.
- 'pc' -> 'PC'
- ground plane had a width of 0.1 => ground pads had only very thin
  connections to ground plane
Parts:
- U$3: value pc -> PC
Changed lines of the file:
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@@
 <layer number="21" name="tPlace" color="7" fill="1" visible="no" active="yes"/>
 <layer number="22" name="bPlace" color="7" fill="1" visible="no" active="yes"/>
-<layer number="23" name="tOrigins" color="7" fill="1" visible="no" active="yes"/>
-<layer number="24" name="bOrigins" color="7" fill="1" visible="no" active="yes"/>
+<layer number="23" name="tOrigins" color="7" fill="1" visible="yes" active="yes"/>
+<layer number="24" name="bOrigins" color="7" fill="1" visible="yes" active="yes"/>
 <layer number="25" name="tNames" color="7" fill="1" visible="no" active="yes"/>
 <layer number="26" name="bNames" color="7" fill="1" visible="no" active="yes"/>
@@
 <element name="L7" library="SparkFun-Passives" package="NPI75C" value="" x="47" y="22.5" rot="R270"/>
 <element name="U$1" library="sam_icons" package="ARROW" value="" x="91.875" y="24.5" rot="R180"/>
-<element name="U$3" library="sam_icons" package="POWER_TEXT" value="pc" x="24.5" y="36.75" rot="R90"/>
+<element name="U$3" library="sam_icons" package="POWER_TEXT" value="PC" x="24.5" y="36.75" rot="R90"/>
 <element name="U$6" library="sam_icons" package="POWER_TEXT" value="AUDIO" x="49" y="36.75" rot="R90"/>
 <element name="U$7" library="sam_icons" package="HOME" value="" x="128.625" y="12.25" rot="R90"/>
@@
 <vertex x="2" y="11"/>
 </polygon>
-<polygon width="0.1" layer="1">
+<polygon width="0.3048" layer="1">
 <vertex x="22" y="2"/>
 <vertex x="22" y="6"/>
@@
 <via x="54" y="28" extent="1-16" drill="0.6"/>
 <via x="72" y="29" extent="1-16" drill="0.6"/>
-<polygon width="0.254" layer="16">
+<polygon width="0.3048" layer="16">
 <vertex x="22" y="47"/>
 <vertex x="212" y="47"/>
@@
 <via x="86" y="40" extent="1-16" drill="0.6"/>
 <via x="86" y="27" extent="1-16" drill="0.6"/>
+<wire x1="40.07" y1="11.78" x2="38.87" y2="11.83" width="0" layer="19" extent="1-1"/>
+<wire x1="42.5" y1="11.5" x2="42.47" y2="11.78" width="0" layer="19" extent="1-1"/>
+<wire x1="41.22" y1="13.18" x2="41.27" y2="11.78" width="0" layer="19" extent="1-1"/>
 </signal>
 <signal name="N$1">
