File: AXremote_circuit/receiver.brd (EAGLE design)
At the start: 50 x 50 mm, 67 parts, among them Q1 16MHz, Q2 MOSFET-NCHANNELBSS138, Q3 MOSFET-NCHANNELBSS138, U1 AX8052F143HS, X1 MINI-USB-SCHIELD-32005-201

Commit message: Add Aperture Logo to receiver.
Parts:
- added U$11: (no value), sam_icons:APERTURE_LOGO_BLACK
Changed lines of the file:
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@@
 <grid distance="1" unitdist="mm" unit="mm" style="lines" multiple="1" display="yes" altdistance="0.5" altunitdist="mm" altunit="mm"/>
 <layers>
-<layer number="1" name="Top" color="4" fill="1" visible="yes" active="yes"/>
+<layer number="1" name="Top" color="4" fill="1" visible="no" active="yes"/>
 <layer number="2" name="Route2" color="1" fill="3" visible="no" active="no"/>
 <layer number="3" name="Route3" color="4" fill="3" visible="no" active="no"/>
@@
 <layer number="15" name="Route15" color="4" fill="6" visible="no" active="no"/>
 <layer number="16" name="Bottom" color="1" fill="1" visible="yes" active="yes"/>
-<layer number="17" name="Pads" color="2" fill="1" visible="yes" active="yes"/>
-<layer number="18" name="Vias" color="2" fill="1" visible="yes" active="yes"/>
-<layer number="19" name="Unrouted" color="6" fill="1" visible="yes" active="yes"/>
-<layer number="20" name="Dimension" color="15" fill="1" visible="yes" active="yes"/>
-<layer number="21" name="tPlace" color="7" fill="1" visible="yes" active="yes"/>
-<layer number="22" name="bPlace" color="7" fill="1" visible="yes" active="yes"/>
-<layer number="23" name="tOrigins" color="15" fill="1" visible="yes" active="yes"/>
+<layer number="17" name="Pads" color="2" fill="1" visible="no" active="yes"/>
+<layer number="18" name="Vias" color="2" fill="1" visible="no" active="yes"/>
+<layer number="19" name="Unrouted" color="6" fill="1" visible="no" active="yes"/>
+<layer number="20" name="Dimension" color="15" fill="1" visible="no" active="yes"/>
+<layer number="21" name="tPlace" color="7" fill="1" visible="no" active="yes"/>
+<layer number="22" name="bPlace" color="7" fill="1" visible="no" active="yes"/>
+<layer number="23" name="tOrigins" color="15" fill="1" visible="no" active="yes"/>
 <layer number="24" name="bOrigins" color="15" fill="1" visible="yes" active="yes"/>
 <layer number="25" name="tNames" color="7" fill="1" visible="no" active="yes"/>
@@
 <layer number="49" name="Reference" color="7" fill="1" visible="yes" active="yes"/>
 <layer number="50" name="dxf" color="7" fill="1" visible="no" active="no"/>
-<layer number="51" name="tDocu" color="7" fill="1" visible="yes" active="yes"/>
+<layer number="51" name="tDocu" color="7" fill="1" visible="no" active="yes"/>
 <layer number="52" name="bDocu" color="7" fill="1" visible="yes" active="yes"/>
 <layer number="53" name="tGND_GNDA" color="7" fill="9" visible="no" active="no"/>
@@
 <element name="C6" library="resistor" package="C0603" value="0" x="22.71" y="14.99" rot="R90"/>
 <element name="C7" library="resistor" package="C0603" value="0" x="22.71" y="8.87" rot="R90"/>
-<element name="Q1" library="crystal" package="SM49" value="16MHz" x="29.39" y="21.71">
-<attribute name="OC_NEWARK" value="unknown" x="29.39" y="21.71" size="1.778" layer="27" display="off"/>
-<attribute name="MPN" value="" x="29.39" y="21.71" size="1.778" layer="27" display="off"/>
-<attribute name="MF" value="" x="29.39" y="21.71" size="1.778" layer="27" display="off"/>
-<attribute name="OC_FARNELL" value="unknown" x="29.39" y="21.71" size="1.778" layer="27" display="off"/>
-</element>
+<element name="Q1" library="crystal" package="SM49" value="16MHz" x="29.39" y="21.71"/>
 <element name="U$1" library="sam_eagle_parts" package="TSOT-23" value="LT1761" x="37.4" y="36.8"/>
 <element name="C1" library="resistor" package="153CLV-0405" value="10uF" x="26" y="27.9" rot="R90"/>
@@
 <attribute name="PROD_ID" value="TRANS-00830" x="41.5" y="42.1" size="1.778" layer="27" rot="R270" display="off"/>
 </element>
+<element name="U$11" library="sam_icons" package="APERTURE_LOGO_BLACK" value="" x="28" y="11" rot="MR0"/>
 </elements>
 <signals>

Commit message: Receiver: Minor fix, export for production.
Parts:
- moved PWR_LED 0.32 mm to (47.0, 21.8)
- moved R16 0.10 mm to (26.4, 23.4)
Routing:
- net GND: track 31.3 -> 37.9 mm, vias 80 -> 83
- net SPI_!INT: track 41.5 -> 40.9 mm

Commit message: working on IR
Parts:
- R15, R18: value 100 -> 10k
Changed lines of the file:
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@@
 </element>
 <element name="R17" library="resistor" package="R0603" value="10k" x="41.4" y="15.4" rot="R90"/>
-<element name="R18" library="resistor" package="R0603" value="100" x="32.4" y="32.6" rot="R180"/>
+<element name="R18" library="resistor" package="R0603" value="10k" x="32.4" y="32.6" rot="R180"/>
 <element name="R11" library="resistor" package="R0603" value="100" x="47.7" y="42.2" rot="R270"/>
 <element name="R13" library="resistor" package="R0603" value="100" x="45.5" y="42.9"/>
@@
 <element name="R10" library="resistor" package="R0603" value="10k" x="40.4" y="4.4" rot="R180"/>
 <element name="U$10" library="sam" package="TACTILE_SWITCH_FSM2JSMA" value="SWITCHSMD" x="26.2" y="36.8" rot="R180"/>
-<element name="R15" library="resistor" package="R0603" value="100" x="26.4" y="32.6"/>
+<element name="R15" library="resistor" package="R0603" value="10k" x="26.4" y="32.6"/>
 <element name="JP1" library="jumper" package="JP2" value="" x="45.9" y="1.7" rot="R180"/>
 <element name="X2" library="axsem_osc_v1-2" package="X3225" value="" x="29.5" y="22.5" rot="R270"/>
